File: 5wy19/can.kicad_sch (KiCad schematic)
At the start: 0 parts

Commit message: Finished most of the subsystems
-- MCU finished
-- Flash finished
-- Power Supply finished
-- I/O Drivers finished
-- CANBUS finished
-- Knock Control finished
-- Connector finished
-- Ignition Driver finished
-- Sensor Logic mostly finished
-- Logic ICs need some work
Parts:
- added C77, C88: 100nf, symbol Device:C_Small
- added IC11: PCA82C250, symbol SIMK43:PCA82C250
- added L1: B82793, symbol Device:L_Coupled_Small_1324
- added R150, R156: 60.4R, symbol Device:R_Small
- added R152: 21.2k, symbol Device:R_Small
Connections:
- new net: IC11.7 (CANH), L1.1
- new net: IC11.6 (CANL), L1.2
- new net: IC11.8 (Rs), R152.2
- new net: C88.2, R150.1, R156.1
- new net 5V: C77.1, IC11.3 (Vcc)
- new net CAN High: L1.3, R150.2
- new net CAN Low: L1.4, R156.2
- new net CAN RXD: IC11.4 (RXD)
- new net CAN TX OUT: IC11.1 (TXD)
- new net GND: C77.2, C88.1, IC11.2 (GND), R152.1
- no-connect marks 0 -> 1
Other:
- title: (none) -> SMIK43 5WY19 Rev. Eng

Commit message: Final schematic (except maybe some oversights)
Parts:
- renumbered R156 to R150, R150 to R156
Connections:
- net CAN High: now also L1.4, R150.2; no longer L1.3, R156.2
- net CAN Low: now also L1.3, R156.2; no longer L1.4, R150.2
Changed lines of the file:
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@@
 		)
 	)
-	(global_label "CAN High"
+	(global_label "CAN Low"
 		(shape input)
 		(at 189.23 91.44 0)
@@
 		)
 		(property "Intersheetrefs" "${INTERSHEET_REFS}"
-			(at 201.1052 91.44 0)
+			(at 200.3795 91.44 0)
+			(effects
+				(font
+					(size 1.27 1.27)
+				)
+				(justify left)
+				(hide yes)
+			)
+		)
+	)
+	(global_label "CAN High"
+		(shape input)
+		(at 189.23 109.22 0)
+		(fields_autoplaced yes)
+		(effects
+			(font
+				(size 1.27 1.27)
+			)
+			(justify left)
+		)
+		(property "Intersheetrefs" "${INTERSHEET_REFS}"
+			(at 201.1052 109.22 0)
 			(effects
 				(font
@@
 				)
 				(justify right)
-				(hide yes)
-			)
-		)
-	)
-	(global_label "CAN Low"
-		(shape input)
-		(at 189.23 109.22 0)
-		(fields_autoplaced yes)
-		(effects
-			(font
-				(size 1.27 1.27)
-			)
-			(justify left)
-		)
-		(property "Intersheetrefs" "${INTERSHEET_REFS}"
-			(at 200.3795 109.22 0)
-			(effects
-				(font
-					(size 1.27 1.27)
-				)
-				(justify left)
 				(hide yes)
 			)
@@
 		(on_board yes)
 		(dnp no)
-		(property "Reference" "R150"
+		(property "Reference" "R156"
 			(at 180.594 94.742 90)
 			(effects
@@
 			(project "5wy19_converted"
 				(path "/abd366a8-4ac6-4ee7-9079-ac453affd4f2/bcea594f-5802-461c-b871-25b4e6f18846"
-					(reference "R150")
+					(reference "R156")
 					(unit 1)
 				)
@@
 		(on_board yes)
 		(dnp no)
-		(property "Reference" "R156"
+		(property "Reference" "R150"
 			(at 180.848 106.172 90)
 			(effects
@@
 			(project "5wy19_converted"
 				(path "/abd366a8-4ac6-4ee7-9079-ac453affd4f2/bcea594f-5802-461c-b871-25b4e6f18846"
-					(reference "R156")
+					(reference "R150")
 					(unit 1)
 				)
